Commit message: Recalibrate Gripper G2 assets, support random spawns in Pick & Place RL, and release v0.3.6

File: assets/urdf/gripper_g2/gripper_g2.urdf (robot description, URDF)
Before this commit: robot gripper_g2, 8 links, 8 joints
Joints:
- joint drive_joint: origin xyz=0 0.035 0.059098 rpy=0 0 0 -> xyz=0 0.035 0.0606 rpy=0 0 0
- joint joint_tcp: origin xyz=0 0 0.172 rpy=0 0 0 -> xyz=0 0 0.1735 rpy=0 0 0
- joint left_inner_knuckle_joint: origin xyz=0 0.02 0.074098 rpy=0 0 0 -> xyz=0 0.02 0.075602 rpy=0 0 0
- joint right_inner_knuckle_joint: origin xyz=0 -0.02 0.074098 rpy=0 0 0 -> xyz=0 -0.02 0.075602 rpy=0 0 0
- joint right_outer_knuckle_joint: origin xyz=0 -0.035 0.059098 rpy=0 0 0 -> xyz=0 -0.035 0.0606 rpy=0 0 0

File: assets/urdf/gripper_g2/gripper_g2_movable_visual.urdf (robot description, URDF)
Before this commit: robot gripper_g2_movable_visual, 9 links, 8 joints
Joints:
- joint drive_joint: origin xyz=0 0.035 0.059098 rpy=0 0 0 -> xyz=0 0.035 0.0606 rpy=0 0 0
- joint joint_tcp: origin xyz=0 0 0.172 rpy=0 0 0 -> xyz=0 0 0.1735 rpy=0 0 0
- joint left_inner_knuckle_joint: origin xyz=0 0.02 0.074098 rpy=0 0 0 -> xyz=0 0.02 0.075602 rpy=0 0 0
- joint right_inner_knuckle_joint: origin xyz=0 -0.02 0.074098 rpy=0 0 0 -> xyz=0 -0.02 0.075602 rpy=0 0 0
- joint right_outer_knuckle_joint: origin xyz=0 -0.035 0.059098 rpy=0 0 0 -> xyz=0 -0.035 0.0606 rpy=0 0 0

File: assets/urdf/uf850/uf850_g2_movable_visual.urdf (robot description, URDF)
Before this commit: robot uf850_g2_movable_visual, 16 links, 15 joints
Joints:
- joint drive_joint: origin xyz=0 0.035 0.059098 rpy=0 0 0 -> xyz=0 0.035 0.0606 rpy=0 0 0
- joint joint_tcp: origin xyz=0 0 0.172 rpy=0 0 0 -> xyz=0 0 0.1735 rpy=0 0 0
- joint left_inner_knuckle_joint: origin xyz=0 0.02 0.074098 rpy=0 0 0 -> xyz=0 0.02 0.075602 rpy=0 0 0
- joint right_inner_knuckle_joint: origin xyz=0 -0.02 0.074098 rpy=0 0 0 -> xyz=0 -0.02 0.075602 rpy=0 0 0
- joint right_outer_knuckle_joint: origin xyz=0 -0.035 0.059098 rpy=0 0 0 -> xyz=0 -0.035 0.0606 rpy=0 0 0

File: assets/urdf/uf850/uf850_g2_visual.urdf (robot description, URDF)
Before this commit: robot uf850_g2_visual, 17 links, 16 joints
Joints:
- joint drive_joint: origin xyz=0 0.035 0.059098 rpy=0 0 0 -> xyz=0 0.035 0.0606 rpy=0 0 0
- joint joint_tcp: origin xyz=0 0 0.172 rpy=0 0 0 -> xyz=0 0 0.1735 rpy=0 0 0
- joint left_inner_knuckle_joint: origin xyz=0 0.02 0.074098 rpy=0 0 0 -> xyz=0 0.02 0.075602 rpy=0 0 0
- joint right_inner_knuckle_joint: origin xyz=0 -0.02 0.074098 rpy=0 0 0 -> xyz=0 -0.02 0.075602 rpy=0 0 0
- joint right_outer_knuckle_joint: origin xyz=0 -0.035 0.059098 rpy=0 0 0 -> xyz=0 -0.035 0.0606 rpy=0 0 0

File: assets/urdf/xarm5/xarm5_1305_g2_movable_visual.urdf (robot description, URDF)
Before this commit: robot xarm5_1305_g2_movable_visual, 15 links, 14 joints
Joints:
- joint drive_joint: origin xyz=0 0.035 0.059098 rpy=0 0 0 -> xyz=0 0.035 0.0606 rpy=0 0 0
- joint joint_tcp: origin xyz=0 0 0.172 rpy=0 0 0 -> xyz=0 0 0.1735 rpy=0 0 0
- joint left_inner_knuckle_joint: origin xyz=0 0.02 0.074098 rpy=0 0 0 -> xyz=0 0.02 0.075602 rpy=0 0 0
- joint right_inner_knuckle_joint: origin xyz=0 -0.02 0.074098 rpy=0 0 0 -> xyz=0 -0.02 0.075602 rpy=0 0 0
- joint right_outer_knuckle_joint: origin xyz=0 -0.035 0.059098 rpy=0 0 0 -> xyz=0 -0.035 0.0606 rpy=0 0 0

File: assets/urdf/xarm5/xarm5_1305_g2_visual.urdf (robot description, URDF)
Before this commit: robot xarm5_1305_g2_visual, 16 links, 15 joints
Joints:
- joint drive_joint: origin xyz=0 0.035 0.059098 rpy=0 0 0 -> xyz=0 0.035 0.0606 rpy=0 0 0
- joint joint_tcp: origin xyz=0 0 0.172 rpy=0 0 0 -> xyz=0 0 0.1735 rpy=0 0 0
- joint left_inner_knuckle_joint: origin xyz=0 0.02 0.074098 rpy=0 0 0 -> xyz=0 0.02 0.075602 rpy=0 0 0
- joint right_inner_knuckle_joint: origin xyz=0 -0.02 0.074098 rpy=0 0 0 -> xyz=0 -0.02 0.075602 rpy=0 0 0
- joint right_outer_knuckle_joint: origin xyz=0 -0.035 0.059098 rpy=0 0 0 -> xyz=0 -0.035 0.0606 rpy=0 0 0

File: assets/urdf/xarm6/xarm6_1305_g2_movable_visual.urdf (robot description, URDF)
Before this commit: robot xarm6_1305_g2_movable_visual, 17 links, 16 joints
Joints:
- joint drive_joint: origin xyz=0 0.035 0.059098 rpy=0 0 0 -> xyz=0 0.035 0.0606 rpy=0 0 0
- joint joint_tcp: origin xyz=0 0 0.172 rpy=0 0 0 -> xyz=0 0 0.1735 rpy=0 0 0
- joint left_inner_knuckle_joint: origin xyz=0 0.02 0.074098 rpy=0 0 0 -> xyz=0 0.02 0.075602 rpy=0 0 0
- joint right_inner_knuckle_joint: origin xyz=0 -0.02 0.074098 rpy=0 0 0 -> xyz=0 -0.02 0.075602 rpy=0 0 0
- joint right_outer_knuckle_joint: origin xyz=0 -0.035 0.059098 rpy=0 0 0 -> xyz=0 -0.035 0.0606 rpy=0 0 0

File: assets/urdf/xarm6/xarm6_1305_g2_visual.urdf (robot description, URDF)
Before this commit: robot xarm6_1305_g2_visual, 18 links, 17 joints
Joints:
- joint drive_joint: origin xyz=0 0.035 0.059098 rpy=0 0 0 -> xyz=0 0.035 0.0606 rpy=0 0 0
- joint joint_tcp: origin xyz=0 0 0.172 rpy=0 0 0 -> xyz=0 0 0.1735 rpy=0 0 0
- joint left_inner_knuckle_joint: origin xyz=0 0.02 0.074098 rpy=0 0 0 -> xyz=0 0.02 0.075602 rpy=0 0 0
- joint right_inner_knuckle_joint: origin xyz=0 -0.02 0.074098 rpy=0 0 0 -> xyz=0 -0.02 0.075602 rpy=0 0 0
- joint right_outer_knuckle_joint: origin xyz=0 -0.035 0.059098 rpy=0 0 0 -> xyz=0 -0.035 0.0606 rpy=0 0 0

File: assets/urdf/xarm6/xarm6_with_gripper.urdf (robot description, URDF)
Before this commit: robot xarm6_with_gripper, 17 links, 16 joints
Joints:
- joint drive_joint: origin xyz=0 0.035 0.059098 rpy=0 0 0 -> xyz=0 0.035 0.0606 rpy=0 0 0
- joint joint_tcp: origin xyz=0 0 0.172 rpy=0 0 0 -> xyz=0 0 0.1735 rpy=0 0 0
- joint left_inner_knuckle_joint: origin xyz=0 0.02 0.074098 rpy=0 0 0 -> xyz=0 0.02 0.075602 rpy=0 0 0
- joint right_inner_knuckle_joint: origin xyz=0 -0.02 0.074098 rpy=0 0 0 -> xyz=0 -0.02 0.075602 rpy=0 0 0
- joint right_outer_knuckle_joint: origin xyz=0 -0.035 0.059098 rpy=0 0 0 -> xyz=0 -0.035 0.0606 rpy=0 0 0

File: assets/urdf/xarm7/xarm7_1305_g2_movable_visual.urdf (robot description, URDF)
Before this commit: robot xarm7_1305_g2_movable_visual, 17 links, 16 joints
Joints:
- joint drive_joint: origin xyz=0 0.035 0.059098 rpy=0 0 0 -> xyz=0 0.035 0.0606 rpy=0 0 0
- joint joint_tcp: origin xyz=0 0 0.172 rpy=0 0 0 -> xyz=0 0 0.1735 rpy=0 0 0
- joint left_inner_knuckle_joint: origin xyz=0 0.02 0.074098 rpy=0 0 0 -> xyz=0 0.02 0.075602 rpy=0 0 0
- joint right_inner_knuckle_joint: origin xyz=0 -0.02 0.074098 rpy=0 0 0 -> xyz=0 -0.02 0.075602 rpy=0 0 0
- joint right_outer_knuckle_joint: origin xyz=0 -0.035 0.059098 rpy=0 0 0 -> xyz=0 -0.035 0.0606 rpy=0 0 0

File: assets/urdf/xarm7/xarm7_1305_g2_visual.urdf (robot description, URDF)
Before this commit: robot xarm7_1305_g2_visual, 18 links, 17 joints
Joints:
- joint drive_joint: origin xyz=0 0.035 0.059098 rpy=0 0 0 -> xyz=0 0.035 0.0606 rpy=0 0 0
- joint joint_tcp: origin xyz=0 0 0.172 rpy=0 0 0 -> xyz=0 0 0.1735 rpy=0 0 0
- joint left_inner_knuckle_joint: origin xyz=0 0.02 0.074098 rpy=0 0 0 -> xyz=0 0.02 0.075602 rpy=0 0 0
- joint right_inner_knuckle_joint: origin xyz=0 -0.02 0.074098 rpy=0 0 0 -> xyz=0 -0.02 0.075602 rpy=0 0 0
- joint right_outer_knuckle_joint: origin xyz=0 -0.035 0.059098 rpy=0 0 0 -> xyz=0 -0.035 0.0606 rpy=0 0 0
